File: Hardware/Extension Board/Extension Board.kicad_pcb (KiCad board)
At the start: 2 copper layers, 132.7 x 44.4 mm, 34 parts, among them J1 CNX_LED, J10 MODE, J11 TUNING, J12 I2C, J13 I2C, J14 SPI, J15 SD, J16 TFT, J2 CNX_LED, J3 CNX_LED, J4 CNX_LED, J5 SPARE, J6 ARDUINO_DIGITAL, J7 ARDUINO_COMMS, J8 ARDUINO_ANALOG, J9 NEXT_AGAIN, U1 74HC14

Commit message: Classe Rythlmic opur la gestion du tempo
Routing:
- net MOSI: track 126.5 -> 126.0 mm
Changed lines of the file:
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@@
     (thickness 1.6)
     (drawings 46)
-    (tracks 451)
+    (tracks 449)
     (zones 0)
     (modules 34)
@@
     (descr "JST XH series connector, B4B-XH-AM, with boss (http://www.jst-mfg.com/product/pdf/eng/eXH.pdf), generated with kicad-footprint-generator")
     (tags "connector JST XH vertical boss")
-    (fp_text reference J15 (at 3.81 1.905 270) (layer F.SilkS)
+    (fp_text reference J15 (at 2.54 1.905 270) (layer F.SilkS)
       (effects (font (size 1 1) (thickness 0.15)))
     )
@@
     (descr "JST XH series connector, B8B-XH-AM, with boss (http://www.jst-mfg.com/product/pdf/eng/eXH.pdf), generated with kicad-footprint-generator")
     (tags "connector JST XH vertical boss")
-    (fp_text reference J16 (at 8.75 1.905) (layer F.SilkS)
+    (fp_text reference J16 (at 5.08 1.905) (layer F.SilkS)
       (effects (font (size 1 1) (thickness 0.15)))
     )
@@
     (descr "JST XH series connector, B4B-XH-A (http://www.jst-mfg.com/product/pdf/eng/eXH.pdf), generated with kicad-footprint-generator")
     (tags "connector JST XH vertical")
-    (fp_text reference J10 (at 0 1.905 180) (layer F.SilkS)
+    (fp_text reference J10 (at 3.81 1.905 180) (layer F.SilkS)
       (effects (font (size 1 1) (thickness 0.15)))
     )
@@
     (descr "5-pin Resistor SIP pack")
     (tags R)
-    (fp_text reference RN1 (at 6.35 -2.4) (layer F.SilkS)
+    (fp_text reference RN1 (at 12.7 0 90) (layer F.SilkS)
       (effects (font (size 1 1) (thickness 0.15)))
     )
@@
     (descr "Resistor, Axial_DIN0207 series, Axial, Horizontal, pin pitch=10.16mm, 0.25W = 1/4W, length*diameter=6.3*2.5mm^2, http://cdn-reichelt.de/documents/datenblatt/B400/1_4W%23YAG.pdf")
     (tags "Resistor Axial_DIN0207 series Axial Horizontal pin pitch 10.16mm 0.25W = 1/4W length 6.3mm diameter 2.5mm")
-    (fp_text reference R4 (at 5.08 0) (layer F.SilkS)
+    (fp_text reference R4 (at 3.81 0) (layer F.SilkS)
       (effects (font (size 1 1) (thickness 0.15)))
     )
@@
     (descr "Resistor, Axial_DIN0207 series, Axial, Horizontal, pin pitch=10.16mm, 0.25W = 1/4W, length*diameter=6.3*2.5mm^2, http://cdn-reichelt.de/documents/datenblatt/B400/1_4W%23YAG.pdf")
     (tags "Resistor Axial_DIN0207 series Axial Horizontal pin pitch 10.16mm 0.25W = 1/4W length 6.3mm diameter 2.5mm")
-    (fp_text reference R3 (at 5.08 0) (layer F.SilkS)
+    (fp_text reference R3 (at 3.81 0) (layer F.SilkS)
       (effects (font (size 1 1) (thickness 0.15)))
     )
@@
     (descr "Resistor, Axial_DIN0207 series, Axial, Horizontal, pin pitch=10.16mm, 0.25W = 1/4W, length*diameter=6.3*2.5mm^2, http://cdn-reichelt.de/documents/datenblatt/B400/1_4W%23YAG.pdf")
     (tags "Resistor Axial_DIN0207 series Axial Horizontal pin pitch 10.16mm 0.25W = 1/4W length 6.3mm diameter 2.5mm")
-    (fp_text reference R2 (at 5.08 0) (layer F.SilkS)
+    (fp_text reference R2 (at 3.81 0) (layer F.SilkS)
       (effects (font (size 1 1) (thickness 0.15)))
     )
@@
     (descr "Resistor, Axial_DIN0207 series, Axial, Horizontal, pin pitch=10.16mm, 0.25W = 1/4W, length*diameter=6.3*2.5mm^2, http://cdn-reichelt.de/documents/datenblatt/B400/1_4W%23YAG.pdf")
     (tags "Resistor Axial_DIN0207 series Axial Horizontal pin pitch 10.16mm 0.25W = 1/4W length 6.3mm diameter 2.5mm")
-    (fp_text reference R1 (at 5.08 0) (layer F.SilkS)
+    (fp_text reference R1 (at 3.81 0) (layer F.SilkS)
       (effects (font (size 1 1) (thickness 0.15)))
     )
@@
     (descr "14-lead though-hole mounted DIP package, row spacing 7.62 mm (300 mils), Socket, LongPads")
     (tags "THT DIP DIL PDIP 2.54mm 7.62mm 300mil Socket LongPads")
-    (fp_text reference U1 (at 5.08 7.62 180) (layer F.SilkS)
+    (fp_text reference U1 (at 3.175 0.635 270) (layer F.SilkS)
       (effects (font (size 1 1) (thickness 0.15)))
     )
@@
   (segment (start 92.71 71.16) (end 94.615 71.12) (width 0.25) (layer F.Cu) (net 11) (status 10))
   (segment (start 94.615 71.12) (end 98.385 71.16) (width 0.25) (layer F.Cu) (net 11))
-  (via (at 92.709992 62.865) (size 0.8) (drill 0.4) (layers F.Cu B.Cu) (net 11))
+  (segment (start 99.498004 62.23) (end 92.709992 62.23) (width 0.25) (layer B.Cu) (net 11))
+  (segment (start 99.695 62.426996) (end 99.498004 62.23) (width 0.25) (layer B.Cu) (net 11))
+  (via (at 92.709992 62.23) (size 0.8) (drill 0.4) (layers F.Cu B.Cu) (net 11))
+  (segment (start 81.91782 62.23) (end 92.709992 62.23) (width 0.25) (layer F.Cu) (net 11))
   (segment (start 99.695 68.58) (end 99.695 62.426996) (width 0.25) (layer B.Cu) (net 11))
-  (segment (start 99.695 62.426996) (end 99.498004 62.23) (width 0.25) (layer B.Cu) (net 11))
-  (segment (start 99.498004 62.23) (end 93.344992 62.23) (width 0.25) (layer B.Cu) (net 11))
-  (segment (start 93.344992 62.23) (end 92.709992 62.865) (width 0.25) (layer B.Cu) (net 11))
-  (segment (start 65.53 50.165) (end 69.85282 50.165) (width 0.25) (layer F.Cu) (net 11))
-  (segment (start 92.074992 62.23) (end 92.709992 62.865) (width 0.25) (layer F.Cu) (net 11))
   (segment (start 62.31 46.945) (end 65.53 50.165) (width 0.25) (layer F.Cu) (net 11))
   (segment (start 62.31 45.72) (end 62.31 46.945) (width 0.25) (layer F.Cu) (net 11) (status 10))
+  (segment (start 65.53 50.165) (end 69.85282 50.165) (width 0.25) (layer F.Cu) (net 11))
   (segment (start 69.85282 50.165) (end 81.91782 62.23) (width 0.25) (layer F.Cu) (net 11))
-  (segment (start 81.91782 62.23) (end 92.074992 62.23) (width 0.25) (layer F.Cu) (net 11))
   (via (at 97.78998 64.77) (size 0.8) (drill 0.4) (layers F.Cu B.Cu) (net 12))
   (segment (start 97.78998 67.31002) (end 97.78998 64.77) (width 0.25) (layer B.Cu) (net 12))

Commit message: update shematics
Parts:
- removed the J16 at (121.9, 68.6)
- added J5: CNX_LED, Connector_JST:JST_XH_B2B-XH-A_1x02_P2.50mm_Vertical, F.Cu at (117.5, 16.5)
- added R11: 200, Resistor_THT:R_Axial_DIN0207_L6.3mm_D2.5mm_P10.16mm_Horizontal, F.Cu at (102.3, 9.20)
- added R12: 200, Resistor_THT:R_Axial_DIN0207_L6.3mm_D2.5mm_P10.16mm_Horizontal, F.Cu at (102.3, 13.2)
- added TP3: TestPoint_Flag, TestPoint:TestPoint_Loop_D2.54mm_Drill1.5mm_Beaded, F.Cu at (128.1, 9.70)
- added U2: LM7806_TO220, Package_TO_SOT_THT:TO-220-3_Vertical, F.Cu at (117.2, 11.1)
- added U3: LM7812_TO220, Package_TO_SOT_THT:TO-220-3_Vertical, F.Cu at (103.9, 19.2)
- J15: value SD -> CNX_LED; footprint Connector_JST:JST_XH_B4B-XH-AM_1x04_P2.50mm_Vertical -> Connector_JST:JST_XH_B2B-XH-A_1x02_P2.50mm_Vertical
- moved J15 66.6 mm to (126.9, 16.5), turned to 0 degrees
- moved J8 17.1 mm to (132.1, 78.1), turned to 0 degrees
- moved J7 13.3 mm to (83.8, 79.4), turned to 0 degrees
- renumbered J5 to J16
Connections:
- J15 pad 1: D17 -> VCC
- J15 pad 2: MOSI -> Net-(J15-Pad2)
- J16 pad 2: Net-(J5-Pad2) -> Net-(J16-Pad2)
- J6 pad 15: Net-(J6-Pad15) -> D35
- J6 pad 17: Net-(J6-Pad17) -> D37
- J7 pad 1: SCL -> Net-(J7-Pad1)
- J7 pad 2: SDA -> Net-(J7-Pad2)
- J7 pad 3: D19 -> D18
- J7 pad 4: D18 -> D19
- J7 pad 5: D17 -> SDA
- J7 pad 6: Net-(J7-Pad6) -> SCL
- J8 pad 2: A14 -> Net-(J8-Pad2)
- J8 pad 4: A12 -> Net-(J8-Pad4)
- J8 pad 5: Net-(J8-Pad5) -> A12
- J8 pad 7: Net-(J8-Pad7) -> A14
- R1 pad 1: Net-(J1-Pad2) -> Net-(J15-Pad2)
- R10 pad 1: /TFT_LED -> Net-(R10-Pad1)
- R9 pad 1: /TFT_LED -> Net-(R9-Pad1)
- TP1 pad 1: VCC -> Net-(TP1-Pad1)
- TP2 pad 1: GND -> Net-(TP2-Pad1)
Routing:
- net Net-(J7-Pad2): track 0.00 -> 10.7 mm
- net D17: track 10.7 -> 0.00 mm

Commit message: Ajout FootPrint Library MesModules
Parts:
- removed the J1 at (111.8, 44.5)
- removed the J2 at (101.6, 44.5)
- removed the J3 at (91.4, 44.5)
- removed the J4 at (80.0, 44.5)
- removed the J5 at (117.5, 16.5)
- removed the R4 at (74.9, 50.8)
- removed the R9 at (114.3, 78.7)
- added C3: 100uF, Capacitor_THT:CP_Axial_L18.0mm_D8.0mm_P25.00mm_Horizontal, F.Cu at (232.4, 24.1)
- added C4: 2200uF, Capacitor_THT:CP_Axial_L30.0mm_D18.0mm_P35.00mm_Horizontal, F.Cu at (200.0, 14.0)
- added C5: 10uF, Capacitor_THT:CP_Radial_D5.0mm_P2.50mm, F.Cu at (170.8, 53.3)
- added C6: 10uF, Capacitor_THT:CP_Radial_D5.0mm_P2.50mm, F.Cu at (172.1, 64.1)
- added J13: CNX_LAMPS, MesModules:Bloc_de_jonction_CI-MPT_2.54mm_01x02, F.Cu at (152.4, 24.1)
- added J14: CNX_6V, TerminalBlock_Phoenix:TerminalBlock_Phoenix_MKDS-1,5-2-5.08_1x02_P5.08mm_Horizontal, F.Cu at (210.8, 75.6)
- added J9: CNX_POWER, TerminalBlock:TerminalBlock_bornier-2_P5.08mm, F.Cu at (211.5, 57.1)
- added JP1: Jumper, Connector_PinHeader_2.54mm:PinHeader_1x02_P2.54mm_Vertical, F.Cu at (189.9, 29.2)
- added JP2: Jumper, Connector_PinHeader_2.54mm:PinHeader_1x02_P2.54mm_Vertical, F.Cu at (170.2, 28.6)
- added R11: 3k3, Resistor_THT:R_Axial_DIN0207_L6.3mm_D2.5mm_P10.16mm_Horizontal, F.Cu at (174.6, 80.0)
- added TP4: TestPoint 12V, TestPoint:TestPoint_Loop_D2.54mm_Drill1.5mm_Beaded, F.Cu at (190.5, 78.7)
- J15: value CNX_LED -> CNX_12V; footprint Connector_JST:JST_XH_B2B-XH-A_1x02_P2.50mm_Vertical -> TerminalBlock_Phoenix:TerminalBlock_Phoenix_MKDS-1,5-2-5.08_1x02_P5.08mm_Horizontal
- R10: value 90k -> 3k3
- R9: renamed from R6; value A CALCULER -> 3M
- TP1: value TestPoint_Flag -> TestPoint GND
- TP2: value TestPoint_Flag -> TestPoint VDD
- TP3: value TestPoint_Flag -> TestPoint 6V
- moved R10 107.7 mm to (211.4, 44.6), turned to 90 degrees
- moved J15 70.6 mm to (191.8, 44.5), turned to 90 degrees
- moved R6 41.4 mm to (143.5, 10.2)
- moved U3 20.9 mm to (83.8, 13.3)
- renumbered J6 to J1, J13 to J16, J7 to J2, J8 to J3, J14 to J4, J10 to J5, J16 to J7, J9 to J8, R5 to R1, R11 to R2, R1 to R3, R2 to R4, R3 to R5, R12 to R6
Connections:
- J11 pad 2: A12 -> /C1
- J15 pad 1: VCC -> +12V
- J15 pad 2: Net-(J15-Pad2) -> GND
- R10 pad 1: Net-(R10-Pad1) -> VCC
- R10 pad 2: VCC -> SDA
- R3 pad 1: Net-(J15-Pad2) -> Net-(J6-Pad5)
- TP1 pad 1: Net-(TP1-Pad1) -> GND
- TP2 pad 1: Net-(TP2-Pad1) -> VDD
- TP3 pad 1: Net-(TP3-Pad1) -> VCC
- U2 pad 1: Net-(U2-Pad1) -> VDD
- U2 pad 2: Net-(U2-Pad2) -> GND
- U2 pad 3: Net-(U2-Pad3) -> VCC
- U3 pad 1: Net-(U3-Pad1) -> VDD
- U3 pad 2: Net-(U3-Pad2) -> GND
- U3 pad 3: Net-(U3-Pad3) -> +12V
Routing:
- net Net-(J6-Pad1): track 16.4 -> 0.00 mm
- net Net-(J5-Pad2): track 0.00 -> 16.4 mm
- net Net-(J6-Pad5): track 0.00 -> 10.3 mm
- net Net-(J6-Pad3): track 10.3 -> 0.00 mm

Commit message: Design carte extension
Parts:
- added C7: 4.7uF, Capacitor_THT:C_Axial_L12.0mm_D7.5mm_P20.00mm_Horizontal, F.Cu at (150.7, 98.8)
- added H3: MountingHole, MountingHole:MountingHole_3.2mm_M3, F.Cu at (78.7, 133.3)
- added H4: MountingHole, MountingHole:MountingHole_3.2mm_M3, F.Cu at (52.1, 59.7)
- added HS1: Heatsink, MesModules:HeatSink_TO-220, F.Cu at (42.7, 42.4)
- added HS2: Heatsink, MesModules:HeatSink_TO-220, F.Cu at (66.1, 42.7)
- added J10: CNX LAMPS, MesModules:Bloc_de_jonction_CI-MPT_2.54mm_01x02, F.Cu at (35.1, 65.3)
- added J17: CNX AUDIO IN, MesModules:Bloc_de_jonction_CI-MPT_2.54mm_01x02, F.Cu at (162.1, 84.6)
- added J18: CNX AUDIO OUT, MesModules:Bloc_de_jonction_CI-MPT_2.54mm_01x02, F.Cu at (194.3, 81.3)
- added J19: CNX AUDIO OUT, MesModules:Bloc_de_jonction_CI-MPT_2.54mm_01x02, F.Cu at (194.3, 88.9)
- added J6: CNX POWER, TerminalBlock_Phoenix:TerminalBlock_Phoenix_MKDS-1,5-2-5.08_1x02_P5.08mm_Horizontal, F.Cu at (35.3, 130.6)
- added JP3: Jumper_3, Connector_PinHeader_2.54mm:PinHeader_1x03_P2.54mm_Vertical, F.Cu at (169.2, 85.1)
- added R12: 10k, Resistor_THT:R_Axial_DIN0207_L6.3mm_D2.5mm_P10.16mm_Horizontal, F.Cu at (173.9, 87.8)
- added R13: 100, Resistor_THT:R_Axial_DIN0207_L6.3mm_D2.5mm_P10.16mm_Horizontal, F.Cu at (184.2, 91.4)
- C4: moved to B.Cu
- J11: value TUNING -> CNX TUNE
- J12, J16: value I2C -> CNX I2C
- J13: value CNX_LAMPS -> CNX_6V; footprint MesModules:Bloc_de_jonction_CI-MPT_2.54mm_01x02 -> TerminalBlock_Phoenix:TerminalBlock_Phoenix_MKDS-1,5-2-5.08_1x02_P5.08mm_Horizontal
- J14: value CNX_6V -> CNX_12V; footprint TerminalBlock_Phoenix:TerminalBlock_Phoenix_MKDS-1,5-2-5.08_1x02_P5.08mm_Horizontal -> TerminalBlock_MetzConnect:TerminalBlock_MetzConnect_Type011_RT05502HBWC_1x02_P5.00mm_Horizontal
- J15: value CNX_12V -> CNX LEDS; footprint TerminalBlock_Phoenix:TerminalBlock_Phoenix_MKDS-1,5-2-5.08_1x02_P5.08mm_Horizontal -> MesModules:HE10-10P-horizontal
- J4: value SPI -> CNX SPI; moved to F.Cu
- J5: value MODE -> CNX MODE
- J7: value SPARE -> CNX SPARE; footprint Connector_JST:JST_XH_B3B-XH-A_1x03_P2.50mm_Vertical -> Connector_JST:JST_XH_B3B-XH-AM_1x03_P2.50mm_Vertical; moved to F.Cu
- J8: value NEXT_AGAIN -> CNX NEXT_AGAIN
- J9: value CNX_POWER -> CNX ON_OFF; footprint TerminalBlock:TerminalBlock_bornier-2_P5.08mm -> Connector_JST:JST_XH_B2B-XH-A_1x02_P2.50mm_Vertical
- R7, R8: value 4.7k -> 3k3
- R9: footprint Resistor_THT:R_Axial_DIN0411_L9.9mm_D3.6mm_P20.32mm_Horizontal -> Resistor_THT:R_Axial_DIN0414_L11.9mm_D4.5mm_P20.32mm_Horizontal
- TP1: value TestPoint GND -> TestPoint VDD
- TP2: value TestPoint VDD -> TestPoint GND
- U1: value 74HC14 -> LM7812_TO220; footprint Package_DIP:DIP-14_W7.62mm_Socket_LongPads -> Package_TO_SOT_THT:TO-220-3_Vertical
- U3: value LM7812_TO220 -> 74HC14; footprint Package_TO_SOT_THT:TO-220-3_Vertical -> Package_DIP:DIP-14_W7.62mm_Socket_LongPads
- moved C3 200.5 mm to (40.6, 82.5), turned to 0 degrees
- moved H2 164.9 mm to (174.0, 132.1)
- moved C4 163.6 mm to (44.7, 65.3), turned to 270 degrees
- moved J9 163.2 mm to (66.3, 131.8), turned to 0 degrees
- moved TP4 158.9 mm to (33.8, 105.0), turned to 0 degrees
- moved RN1 152.4 mm to (185.4, 49.5), turned to 270 degrees
- moved R10 147.0 mm to (65.5, 63.2), turned to 270 degrees
- moved C6 132.0 mm to (43.2, 92.7), turned to 0 degrees
- moved R2 127.6 mm to (176.0, 113.3), turned to 180 degrees
- moved TP3 127.1 mm to (33.8, 95.0)
- moved J5 126.5 mm to (193.8, 59.7), turned to 90 degrees
- moved C5 123.6 mm to (53.6, 92.7), turned to 0 degrees
- moved TP2 118.9 mm to (33.8, 85.6), turned to 0 degrees
- moved R11 116.9 mm to (58.9, 63.2), turned to 270 degrees
- moved R5 113.3 mm to (176.0, 123.2), turned to 180 degrees
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Connections:
- net /C1 renamed /Connectors/C1
- J1 pad 10: Net-(J1-Pad10) -> (no net)
- J1 pad 11: Net-(J1-Pad11) -> (no net)
- J1 pad 12: Net-(J1-Pad12) -> (no net)
- J1 pad 13: D33 -> (no net)
- J1 pad 14: Net-(J1-Pad14) -> (no net)
- J1 pad 15: D35 -> (no net)
- J1 pad 16: Net-(J1-Pad16) -> (no net)
- J1 pad 18: Net-(J1-Pad18) -> (no net)
- J1 pad 19: Net-(J1-Pad19) -> D23
- J1 pad 20: D38 -> (no net)
- J1 pad 21: Net-(J1-Pad21) -> D25
- J1 pad 22: D40 -> D42
- J1 pad 23: Net-(J1-Pad23) -> D27
- J1 pad 24: D42 -> (no net)
- J1 pad 27: Net-(J1-Pad27) -> D47
- J1 pad 3: D23 -> (no net)
- J1 pad 30: Net-(J1-Pad30) -> (no net)
- J1 pad 33: Net-(J1-Pad33) -> (no net)
- J1 pad 4: Net-(J1-Pad4) -> (no net)
- J1 pad 5: D25 -> (no net)
- J1 pad 6: Net-(J1-Pad6) -> (no net)
- J1 pad 7: D27 -> (no net)
- J1 pad 8: Net-(J1-Pad8) -> (no net)
- J1 pad 9: D29 -> (no net)
- J14 pad 1: VCC -> +12V
- J15 pad 1: +12V -> Net-(J15-Pad1)
- J15 pad 2: GND -> VCC
- J2 pad 1: Net-(J2-Pad1) -> (no net)
- J2 pad 2: Net-(J2-Pad2) -> (no net)
- J3 pad 1: Net-(J3-Pad1) -> (no net)
- J3 pad 2: Net-(J3-Pad2) -> (no net)
- J3 pad 3: Net-(J3-Pad3) -> (no net)
- J3 pad 4: Net-(J3-Pad4) -> (no net)
- J3 pad 6: Net-(J3-Pad6) -> (no net)
- J3 pad 8: Net-(J3-Pad8) -> (no net)
- J4 pad 2: D33 -> D42
- J9 pad 1: GND -> Net-(J6-Pad2)
- J9 pad 2: Net-(J10-Pad1) -> VDD
- R1 pad 1: Net-(J6-Pad1) -> Net-(J15-Pad1)
- R1 pad 2: D49 -> D45
- R2 pad 1: Net-(J6-Pad3) -> Net-(J15-Pad3)
- R2 pad 2: D35 -> D47
- R3 pad 1: Net-(J6-Pad5) -> Net-(J15-Pad5)
- R3 pad 2: D44 -> D49
- R4 pad 1: Net-(J6-Pad7) -> Net-(J15-Pad7)
- R5 pad 1: Net-(J6-Pad9) -> Net-(J15-Pad9)
- R5 pad 2: D45 -> D44
- RN1 pad 5: Net-(RN1-Pad5) -> (no net)
- TP1 pad 1: GND -> VDD
- TP2 pad 1: VDD -> GND
- U1 pad 1: Net-(C1-Pad1) -> VDD
- U1 pad 2: D19 -> GND
- U1 pad 3: Net-(C2-Pad1) -> +12V
- U3 pad 1: VDD -> Net-(C1-Pad1)
- U3 pad 2: GND -> D19
- U3 pad 3: +12V -> Net-(C2-Pad1)
Routing:
- net VCC: track 319.3 -> 0.00 mm
- net GND: track 285.1 -> 0.00 mm, vias 2 -> 0
- net MOSI: track 126.0 -> 0.00 mm, vias 4 -> 0
- net SCL: track 112.7 -> 0.00 mm
- net SDA: track 105.8 -> 0.00 mm
- net MISO: track 84.0 -> 0.00 mm, vias 1 -> 0
- net SCK: track 83.6 -> 0.00 mm
- net D19: track 73.3 -> 0.00 mm
- net D18: track 65.7 -> 0.00 mm
- net D27: track 65.4 -> 0.00 mm, vias 2 -> 0
- net D25: track 64.2 -> 0.00 mm, vias 2 -> 0
- net D23: track 63.1 -> 0.00 mm, vias 2 -> 0
- net A12: track 58.2 -> 0.00 mm, vias 1 -> 0
- net D46: track 45.8 -> 0.00 mm, vias 1 -> 0
- net Net-(C1-Pad1): track 44.1 -> 0.00 mm
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Other:
- board size 132.7 x 44.4 mm -> 170 x 100 mm
- board text removed: "5V"
- board text removed: "GND"
- board text removed: "LEDs"
- board text removed: "SPARE"
