File: Hardware/Extension Board/Extension Board.kicad_pcb (KiCad board)
At the start: 2 copper layers, 170 x 100 mm, 56 parts, among them J1 ARDUINO_DIGITAL, J10 CNX LAMPS, J11 CNX TUNE, J12 CNX I2C, J13 CNX_6V, J14 CNX_12V, J15 CNX LEDS, J16 CNX I2C, J17 CNX AUDIO IN, J18 CNX AUDIO OUT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

Commit message: début du routage
Parts:
- removed J18: CNX AUDIO OUT, MesModules:Bloc_de_jonction_CI-MPT_2.54mm_01x02
- removed JP3: Jumper_3, Connector_PinHeader_2.54mm:PinHeader_1x03_P2.54mm_Vertical
- HS1, HS2, U1, U2: moved to B.Cu
- J11: value CNX TUNE -> TUNE
- J12, J16: value CNX I2C -> BUS I2C
- J13: value CNX_6V -> CNX 6V
- J14: value CNX_12V -> CNX 12V
- J17: value CNX AUDIO IN -> AUDIO IN
- J19: value CNX AUDIO OUT -> AUDIO OUT
- J3: footprint Connector_PinHeader_2.54mm:PinHeader_1x08_P2.54mm_Vertical -> Connector_PinHeader_2.54mm:PinHeader_1x06_P2.54mm_Vertical
- J4: value CNX SPI -> BUS SPI
- J5: value CNX MODE -> MODE
- J7: value CNX SPARE -> I/O SPARE
- J8: value CNX NEXT_AGAIN -> NEXT_AGAIN
- J9: value CNX ON_OFF -> ON_OFF
- TP1: value TestPoint VDD -> V IN; footprint TestPoint:TestPoint_Loop_D2.54mm_Drill1.5mm_Beaded -> TestPoint:TestPoint_Loop_D2.60mm_Drill1.4mm_Beaded
- TP2: value TestPoint GND -> GND; footprint TestPoint:TestPoint_Loop_D2.54mm_Drill1.5mm_Beaded -> TestPoint:TestPoint_Loop_D2.60mm_Drill1.4mm_Beaded
- TP3: value TestPoint 6V -> 6V; footprint TestPoint:TestPoint_Loop_D2.54mm_Drill1.5mm_Beaded -> TestPoint:TestPoint_Loop_D2.60mm_Drill1.4mm_Beaded
- TP4: value TestPoint 12V -> 12V; footprint TestPoint:TestPoint_Loop_D2.54mm_Drill1.5mm_Beaded -> TestPoint:TestPoint_Loop_D2.60mm_Drill1.4mm_Beaded
- moved TP1 162.1 mm to (195.6, 86.4)
- moved TP2 162.1 mm to (195.6, 95.0)
- moved TP3 162.0 mm to (195.6, 102.9)
- moved TP4 161.9 mm to (195.6, 111.5)
- moved J11 103.1 mm to (55.9, 57.9), turned to 180 degrees
- moved J9 92.0 mm to (83.1, 41.4)
- moved R1 68.1 mm to (161.8, 43.4)
- moved R2 68.1 mm to (161.8, 46.7)
- moved R3 68.1 mm to (161.8, 50.0)
- moved R4 68.1 mm to (161.8, 53.3)
- moved R5 68.1 mm to (161.8, 56.6)
- moved J19 45.4 mm to (179.6, 46.0), turned to 180 degrees
- moved J7 41.2 mm to (74.9, 82.5)
- moved J6 40.6 mm to (75.2, 122.9)
- moved H3 37.9 mm to (41.7, 125.5)
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Connections:
- net D23 renamed D39
- net D25 renamed D41
- net D27 renamed D43
- J1 pad 17: D37 -> (no net)
- J1 pad 20: (no net) -> D40
- J1 pad 22: D42 -> (no net)
- J1 pad 30: (no net) -> D36
- J17 pad 1: Net-(J17-Pad1) -> (no net)
- J17 pad 2: Net-(J17-Pad2) -> Net-(C7-Pad1)
- J19 pad 1: GND -> Net-(J19-Pad1)
- J19 pad 2: Net-(J19-Pad2) -> GND
- J3 pad 3: (no net) -> A12
- J3 pad 5: A12 -> A14
- J4 pad 2: D42 -> D36
- R13 pad 1: Net-(J19-Pad2) -> Net-(J19-Pad1)
- R6 pad 2: D37 -> D40
Routing:
- net D39: track 0.00 -> 97.3 mm, vias 0 -> 1
- net D41: track 0.00 -> 94.6 mm, vias 0 -> 1
- net D43: track 0.00 -> 91.8 mm, vias 0 -> 1
- net MOSI: track 0.00 -> 37.1 mm, vias 0 -> 1
- net D47: track 1.59 -> 37.3 mm, vias 0 -> 1
- net D45: track 0.00 -> 34.9 mm, vias 0 -> 1
- net D49: track 0.00 -> 32.6 mm, vias 0 -> 1
- net D36: track 0.00 -> 14.9 mm, vias 0 -> 1
- net GND: track 0.00 -> 14.2 mm, vias 0 -> 1
- net SCK: track 0.00 -> 14.1 mm, vias 0 -> 1
- net MISO: track 0.00 -> 10.7 mm, vias 0 -> 1
- net (no net): track 2.54 -> 0.00 mm
Other:
- board size 170 x 100 mm -> 164.2 x 93.3 mm
- net class Default: clearance 0.2 -> 0.3; trace_width 0.25 -> 0.3
- net class Power: clearance 0.2 -> 0.3; trace_width 0.4 -> 0.5
- rule trace_clearance: 0.2 -> 0.3
- board text added: "41 43 45 47 49 51 53 GND"
- board text added: "A10"
- board text added: "C0-C2"
- board text added: "C1-C2"
- board text added: "D16"

Commit message: Routage du PCB
Parts:
- C7: footprint Capacitor_THT:C_Axial_L12.0mm_D7.5mm_P20.00mm_Horizontal -> Capacitor_THT:C_Axial_L17.0mm_D7.0mm_P25.00mm_Horizontal
- J2: footprint Connector_PinHeader_2.54mm:PinHeader_1x06_P2.54mm_Vertical -> Connector_PinHeader_2.54mm:PinHeader_1x04_P2.54mm_Vertical
- R9: footprint Resistor_THT:R_Axial_DIN0414_L11.9mm_D4.5mm_P20.32mm_Horizontal -> Resistor_THT:R_Axial_DIN0309_L9.0mm_D3.2mm_P15.24mm_Horizontal
- moved TP1 112.5 mm to (93.0, 40.1)
- moved H4 43.2 mm to (62.5, 49.0)
- moved H2 29.3 mm to (165.6, 126.7)
- moved TP4 25.1 mm to (195.6, 86.4)
- moved H3 22.4 mm to (64.0, 124.7)
- moved J9 21.8 mm to (61.2, 41.4)
- moved J17 13.7 mm to (153.2, 75.9)
- moved RN1 12.7 mm to (185.9, 62.2), turned to 90 degrees
- moved R7 10.2 mm to (53.3, 121.4), turned to 90 degrees
- moved R8 10.2 mm to (49.5, 121.4), turned to 90 degrees
- moved HS2 9.91 mm to (77.7, 40.4)
- moved U2 9.91 mm to (80.3, 50.0)
- moved U3 9.12 mm to (60.2, 102.4)
- moved J12 7.64 mm to (82.3, 67.1), turned to 180 degrees
- moved J5 7.62 mm to (194.1, 52.1), turned to 270 degrees
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Connections:
- J1 pad 18: (no net) -> D36
- J1 pad 20: D40 -> (no net)
- J1 pad 30: D36 -> D48
- J2 pad 1: (no net) -> D18
- J2 pad 2: (no net) -> D19
- J2 pad 3: D18 -> SDA
- J2 pad 4: D19 -> SCL
- J4 pad 2: D36 -> D48
- J5 pad 2: D43 -> D39
- J5 pad 4: D39 -> D43
- R6 pad 2: D40 -> D36
- RN1 pad 2: D39 -> D43
- RN1 pad 4: D43 -> D39
Routing:
- net GND: track 14.2 -> 543.1 mm, vias 1 -> 6
- net VCC: track 0.00 -> 245.4 mm, vias 0 -> 3
- net A14: track 0.00 -> 147.0 mm, vias 0 -> 2
- net VDD: track 0.00 -> 92.1 mm, vias 0 -> 2
- net Net-(J15-Pad1): track 0.00 -> 88.1 mm, vias 0 -> 2
- net Net-(J15-Pad3): track 0.00 -> 85.3 mm, vias 0 -> 2
- net Net-(J15-Pad5): track 0.00 -> 83.4 mm, vias 0 -> 2
- net Net-(J15-Pad7): track 0.00 -> 82.8 mm, vias 0 -> 2
- net Net-(J15-Pad9): track 0.00 -> 80.5 mm, vias 0 -> 2
- net D46: track 0.00 -> 78.1 mm, vias 0 -> 1
- net D44: track 0.00 -> 75.1 mm, vias 0 -> 1
- net Net-(C2-Pad1): track 0.00 -> 63.4 mm
- net SCL: track 0.00 -> 54.2 mm, vias 0 -> 1
- net SDA: track 0.00 -> 46.8 mm, vias 0 -> 1
- net Net-(C7-Pad2): track 0.00 -> 45.9 mm
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Other:
- board size 164.2 x 93.3 mm -> 164.2 x 94.5 mm
- board text added: "31 33 35 37"
- board text added: "D18"
- board text added: "GND"
- board text removed: "41 43 45 47 49 51 53 GND"
- board text removed: "D16"

Commit message: PCB updated
Parts:
- H1, H2, H3, H4: footprint MountingHole:MountingHole_3.2mm_M3 -> MountingHole:MountingHole_2.7mm_M2.5
- moved R7 1.05 mm to (53.1, 122.4)
- moved R8 1.05 mm to (49.3, 122.4)
Routing:
- net GND: track 543.1 -> 544.6 mm
- net Net-(C1-Pad1): track 32.4 -> 33.8 mm
- net Net-(C2-Pad1): track 63.4 -> 64.7 mm
