File: Hardware/Extension Board/Extension Board.kicad_pcb (KiCad board)
At the start: 2 copper layers, 164.2 x 94.5 mm, 54 parts, among them J1 ARDUINO_DIGITAL, J10 CNX LAMPS, J11 TUNE, J12 BUS I2C, J13 CNX 6V, J14 CNX 12V, J15 CNX LEDS, J16 BUS I2C, J17 AUDIO IN, J19 AUDIO OUT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

Commit message: PCB routing completed
Parts:
- moved J16 6.78 mm to (108.2, 65.0), turned to 180 degrees
- moved H2 1.61 mm to (167.1, 126.2)
- moved TP1 1.05 mm to (92.7, 41.1)
- moved J6 0.97 mm to (75.6, 123.8)
Connections:
- net Net-(J6-Pad2) renamed /Alimentation/VSS
Routing:
- net VCC: track 245.4 -> 456.9 mm, vias 3 -> 7
- net +12V: track 41.1 -> 227.5 mm, vias 3 -> 4
- net /Connectors/C1: track 0.00 -> 121.4 mm, vias 0 -> 2
- net /Alimentation/VSS: track 0.00 -> 100.8 mm, vias 0 -> 2
- net D18: track 0.00 -> 72.0 mm, vias 0 -> 1
- net D19: track 0.00 -> 69.0 mm, vias 0 -> 1
- net GND: track 544.6 -> 602.7 mm, vias 6 -> 11
- net SCL: track 54.2 -> 75.1 mm, vias 1 -> 2
- net SDA: track 46.8 -> 63.0 mm, vias 1 -> 2
- net VDD: track 92.1 -> 104.9 mm, vias 2 -> 3
- net D36: track 6.56 -> 8.98 mm
- net A14: track 147.0 -> 144.7 mm
- net Net-(J7-Pad2): track 43.1 -> 45.0 mm
- net MISO: track 11.1 -> 12.0 mm
- net Net-(J19-Pad1): track 34.1 -> 34.8 mm
Other:
- board text added: "+"
- board text added: "-"
- board text added: "GND D36 VCC"
- board text added: "GND SDA SCL VCC"
- board text added: "VCC D48 MOSI SCK MISO GND"

Commit message: Modèles 3D
Parts:
- moved TP1 0.91 mm to (91.8, 41.1)
- moved J2 0.10 mm to (91.8, 65.5)
Routing:
- net GND: track 602.7 -> 601.4 mm
- net VDD: track 104.9 -> 103.9 mm
Other:
- board text added: "2,032mm = 80 mil"
- board text added: "5,080mm = 200mil"
- board text added: "7,620mm = 300 mil"
