File: Hardware/Extension Board/Connectors.sch (KiCad schematic (older format))
At the start: 25 parts, among them J11 CNX TUNE, J12 CNX I2C, J15 CNX LEDS, J16 CNX I2C, J4 CNX SPI, J5 CNX MODE, J7 CNX SPARE, J8 CNX NEXT_AGAIN, U1 74HC14

Commit message: Design carte extension
Parts:
- renumbered U1 to U3
Connections:
- net D44: now also R5.2; no longer R3.2
- net D45: now also R1.2; no longer R5.2
- net D49: now also R3.2; no longer R1.2
- net D33 renamed D42
- net D35 renamed D47
Changed lines of the file:
@@
 $Descr A4 11693 8268
 encoding utf-8
-Sheet 3 3
+Sheet 3 4
 Title ""
 Date ""
@@
 $EndComp
 Text GLabel 1800 1700 0    50   Input ~ 0
-D44
+D49
 Text GLabel 1800 1800 0    50   Input ~ 0
 D46
@@
 	1800 1800 2000 1800
 Text GLabel 1800 1900 0    50   Input ~ 0
-D45
+D44
 Wire Wire Line
 	1800 1900 2000 1900
 Text GLabel 1800 1500 0    50   Input ~ 0
-D49
+D45
 Wire Wire Line
 	1800 1500 2000 1500
 Wire Wire Line
 	1800 1700 2000 1700
-Text Notes 1600 1750 2    50   ~ 0
+Text Notes 1600 1550 2    50   ~ 0
 PWM
 Text Notes 1600 1850 2    50   ~ 0
@@
 	2300 1600 3100 1600
 Text GLabel 1800 1600 0    50   Input ~ 0
-D35
+D47
 Wire Wire Line
 	1800 1600 2000 1600
@@
 	1350 5950 1350 6800
 Text GLabel 1650 5950 1    50   Input ~ 0
-D33
+D42
 Wire Wire Line
 	1250 6200 1250 6800
@@
 P 8400 4400
 AR Path="/625091A0" Ref="U?"  Part="1"
-AR Path="/624DD375/625091A0" Ref="U1"  Part="1"
-F 0 "U1" H 8550 4300 50  0000 C CNN
+AR Path="/624DD375/625091A0" Ref="U3"  Part="1"
+F 0 "U3" H 8550 4300 50  0000 C CNN
 F 1 "74HC14" H 8500 4200 50  0000 C CNN
 F 2 "Package_DIP:DIP-14_W7.62mm_Socket_LongPads" H 8400 4400 50  0001 C CNN
@@
 P 9600 5800
 AR Path="/625091A6" Ref="U?"  Part="7"
-AR Path="/624DD375/625091A6" Ref="U1"  Part="7"
-F 0 "U1" V 9750 5750 50  0000 L CNN
+AR Path="/624DD375/625091A6" Ref="U3"  Part="7"
+F 0 "U3" V 9750 5750 50  0000 L CNN
 F 1 "74HC14" V 9450 5650 50  0000 L CNN
 F 2 "Package_DIP:DIP-14_W7.62mm_Socket_LongPads" H 9600 5800 50  0001 C CNN
@@
 P 8400 4750
 AR Path="/625091C0" Ref="U?"  Part="2"
-AR Path="/624DD375/625091C0" Ref="U1"  Part="2"
-F 0 "U1" H 8550 4650 50  0000 C CNN
+AR Path="/624DD375/625091C0" Ref="U3"  Part="2"
+F 0 "U3" H 8550 4650 50  0000 C CNN
 F 1 "74HC14" H 8500 4550 50  0000 C CNN
 F 2 "Package_DIP:DIP-14_W7.62mm_Socket_LongPads" H 8400 4750 50  0001 C CNN

Commit message: début du routage
Parts:
- J11: value CNX TUNE -> TUNE
- J12, J16: value CNX I2C -> BUS I2C
- J4: value CNX SPI -> BUS SPI
- J5: value CNX MODE -> MODE
- J7: value CNX SPARE -> I/O SPARE
- J8: value CNX NEXT_AGAIN -> NEXT_AGAIN
Connections:
- net D23 renamed D39
- net D25 renamed D41
- net D27 renamed D43
- net D37 renamed D40
- net D42 renamed D48
Changed lines of the file:
@@
 P 1550 7000
 F 0 "J4" V 1550 6500 50  0000 L CNN
-F 1 "CNX SPI" V 1650 6800 50  0000 L CNN
+F 1 "BUS SPI" V 1650 6800 50  0000 L CNN
 F 2 "Connector_JST:JST_XH_B6B-XH-AM_1x06_P2.50mm_Vertical" H 1550 7000 50  0001 C CNN
 F 3 "~" H 1550 7000 50  0001 C CNN
@@
 	1350 5950 1350 6800
 Text GLabel 1650 5950 1    50   Input ~ 0
-D42
+D48
 Wire Wire Line
 	1250 6200 1250 6800
@@
 AR Path="/624DD375/624E8E5D" Ref="J7"  Part="1"
 F 0 "J7" V 2800 6750 50  0000 L CNN
-F 1 "CNX SPARE" V 2950 6800 50  0000 L CNN
+F 1 "I/O SPARE" V 2950 6800 50  0000 L CNN
 F 2 "Connector_JST:JST_XH_B3B-XH-AM_1x03_P2.50mm_Vertical" H 2800 7000 50  0001 C CNN
 F 3 "~" H 2800 7000 50  0001 C CNN
@@
 	2800 6250 2800 5950
 Text GLabel 2800 5950 1    50   BiDi ~ 0
-D37
+D40
 Text Notes 1100 5500 0    50   ~ 0
 Spare connectors
@@
 AR Path="/624DD375/624FC9A4" Ref="J5"  Part="1"
 F 0 "J5" H 7200 1600 50  0000 R CNN
-F 1 "CNX MODE" H 7350 2100 50  0000 R CNN
+F 1 "MODE" H 7300 2100 50  0000 R CNN
 F 2 "Connector_JST:JST_XH_B4B-XH-A_1x04_P2.50mm_Vertical" H 7150 1900 50  0001 C CNN
 F 3 "~" H 7150 1900 50  0001 C CNN
@@
 $EndComp
 Text GLabel 5500 1900 0    50   Output ~ 0
-D27
+D43
 Text GLabel 5500 1800 0    50   Output ~ 0
-D25
+D41
 Text GLabel 5500 1700 0    50   Output ~ 0
-D23
+D39
 Connection ~ 6400 1700
 Wire Wire Line
@@
 AR Path="/624DD375/625091B5" Ref="J8"  Part="1"
 F 0 "J8" H 10700 4750 50  0000 L CNN
-F 1 "CNX NEXT_AGAIN" H 10400 4300 50  0000 L CNN
+F 1 "NEXT_AGAIN" H 10600 4300 50  0000 L CNN
 F 2 "Connector_JST:JST_XH_B3B-XH-A_1x03_P2.50mm_Vertical" H 10750 4500 50  0001 C CNN
 F 3 "~" H 10750 4500 50  0001 C CNN
@@
 AR Path="/624DD375/6251438B" Ref="J16"  Part="1"
 F 0 "J16" H 10650 1850 50  0000 L CNN
-F 1 "CNX I2C" H 10600 1350 50  0000 L CNN
+F 1 "BUS I2C" H 10600 1350 50  0000 L CNN
 F 2 "Connector_JST:JST_XH_B4B-XH-A_1x04_P2.50mm_Vertical" H 10700 1650 50  0001 C CNN
 F 3 "~" H 10700 1650 50  0001 C CNN
@@
 AR Path="/624DD375/625143AF" Ref="J12"  Part="1"
 F 0 "J12" H 9450 1850 50  0000 L CNN
-F 1 "CNX I2C" H 9400 1350 50  0000 L CNN
+F 1 "BUS I2C" H 9400 1350 50  0000 L CNN
 F 2 "Connector_JST:JST_XH_B4B-XH-A_1x04_P2.50mm_Vertical" H 9500 1650 50  0001 C CNN
 F 3 "~" H 9500 1650 50  0001 C CNN
@@
 AR Path="/624DD375/62538B21" Ref="J11"  Part="1"
 F 0 "J11" H 3600 4100 50  0000 R CNN
-F 1 "CNX TUNE" H 3650 3700 50  0000 R CNN
+F 1 "TUNE" H 3650 3700 50  0000 R CNN
 F 2 "Connector_JST:JST_XH_B3B-XH-A_1x03_P2.50mm_Vertical" H 3550 3900 50  0001 C CNN
 F 3 "~" H 3550 3900 50  0001 C CNN

Commit message: Routage du PCB
Parts:
- R9: footprint Resistor_THT:R_Axial_DIN0414_L11.9mm_D4.5mm_P20.32mm_Horizontal -> Resistor_THT:R_Axial_DIN0309_L9.0mm_D3.2mm_P15.24mm_Horizontal
Connections:
- net D39: now also J5.2 (Pin_2), RN1.4 (R3); no longer J5.4 (Pin_4), RN1.2 (R1)
- net D43: now also J5.4 (Pin_4), RN1.2 (R1); no longer J5.2 (Pin_2), RN1.4 (R3)
- net D40 renamed D36
Changed lines of the file:
@@
 	2800 6250 2800 5950
 Text GLabel 2800 5950 1    50   BiDi ~ 0
-D40
+D36
 Text Notes 1100 5500 0    50   ~ 0
 Spare connectors
@@
 $EndComp
 Text GLabel 5500 1900 0    50   Output ~ 0
-D43
+D39
 Text GLabel 5500 1800 0    50   Output ~ 0
 D41
 Text GLabel 5500 1700 0    50   Output ~ 0
-D39
+D43
 Connection ~ 6400 1700
 Wire Wire Line
@@
 F 0 "R9" V 2050 4150 50  0000 C CNN
 F 1 "3M" V 2150 4150 50  0000 C CNN
-F 2 "Resistor_THT:R_Axial_DIN0414_L11.9mm_D4.5mm_P20.32mm_Horizontal" V 1980 4150 50  0001 C CNN
+F 2 "Resistor_THT:R_Axial_DIN0309_L9.0mm_D3.2mm_P15.24mm_Horizontal" V 1980 4150 50  0001 C CNN
 F 3 "~" H 2050 4150 50  0001 C CNN
 	1    2050 4150
