File: Hardware/Extension Board/Alimentation.sch (KiCad schematic (older format))
At the start: 17 parts, among them J10 CNX_LAMPS, J13 CNX_6V, J14 CNX_12V, J6 CNX POWER, J9 CNX ON_OFF, U2 LM7806_TO220, U3 LM7812_TO220

Commit message: Design carte extension
Parts:
- J10: value CNX_LAMPS -> CNX LAMPS
- renumbered U3 to U1
Changed lines of the file:
@@
 $Descr A4 11693 8268
 encoding utf-8
-Sheet 2 3
+Sheet 2 4
 Title ""
 Date ""
@@
 P 6600 5300
 AR Path="/624D4FF9" Ref="U?"  Part="1"
-AR Path="/624BFCA3/624D4FF9" Ref="U3"  Part="1"
-F 0 "U3" H 6700 5050 50  0000 C CNN
+AR Path="/624BFCA3/624D4FF9" Ref="U1"  Part="1"
+F 0 "U1" H 6700 5050 50  0000 C CNN
 F 1 "LM7812_TO220" H 6600 5451 50  0000 C CNN
 F 2 "Package_TO_SOT_THT:TO-220-3_Vertical" H 6600 5525 50  0001 C CIN
@@
 AR Path="/624BFCA3/624D4FFF" Ref="J10"  Part="1"
 F 0 "J10" H 3600 5700 50  0000 R CNN
-F 1 "CNX_LAMPS" H 3800 5400 50  0000 R CNN
+F 1 "CNX LAMPS" H 3800 5400 50  0000 R CNN
 F 2 "MesModules:Bloc_de_jonction_CI-MPT_2.54mm_01x02" H 3550 5600 50  0001 C CNN
 F 3 "~" H 3550 5600 50  0001 C CNN

Commit message: début du routage
Parts:
- J13: value CNX_6V -> CNX 6V
- J14: value CNX_12V -> CNX 12V
- J9: value CNX ON_OFF -> ON_OFF
- TP1: value TestPoint VDD -> V IN; footprint TestPoint:TestPoint_Loop_D2.54mm_Drill1.5mm_Beaded -> TestPoint:TestPoint_Loop_D2.60mm_Drill1.4mm_Beaded
- TP2: value TestPoint GND -> GND; footprint TestPoint:TestPoint_Loop_D2.54mm_Drill1.5mm_Beaded -> TestPoint:TestPoint_Loop_D2.60mm_Drill1.4mm_Beaded
- TP3: value TestPoint 6V -> 6V; footprint TestPoint:TestPoint_Loop_D2.54mm_Drill1.5mm_Beaded -> TestPoint:TestPoint_Loop_D2.60mm_Drill1.4mm_Beaded
- TP4: value TestPoint 12V -> 12V; footprint TestPoint:TestPoint_Loop_D2.54mm_Drill1.5mm_Beaded -> TestPoint:TestPoint_Loop_D2.60mm_Drill1.4mm_Beaded
Changed lines of the file:
@@
 AR Path="/624BFCA3/624C86D1" Ref="TP2"  Part="1"
 F 0 "TP2" H 4100 3100 50  0000 L CNN
-F 1 "TestPoint GND" H 3950 3200 50  0000 L CNN
-F 2 "TestPoint:TestPoint_Loop_D2.54mm_Drill1.5mm_Beaded" H 4050 3050 50  0001 C CNN
+F 1 "GND" H 3950 3200 50  0000 L CNN
+F 2 "TestPoint:TestPoint_Loop_D2.60mm_Drill1.4mm_Beaded" H 4050 3050 50  0001 C CNN
 F 3 "~" H 4050 3050 50  0001 C CNN
 	1    3850 3050
@@
 AR Path="/624BFCA3/624C86D7" Ref="TP1"  Part="1"
 F 0 "TP1" H 4100 1700 50  0000 L CNN
-F 1 "TestPoint VDD" H 3900 1800 50  0000 L CNN
-F 2 "TestPoint:TestPoint_Loop_D2.54mm_Drill1.5mm_Beaded" H 4000 1650 50  0001 C CNN
+F 1 "V IN" H 3900 1800 50  0000 L CNN
+F 2 "TestPoint:TestPoint_Loop_D2.60mm_Drill1.4mm_Beaded" H 4000 1650 50  0001 C CNN
 F 3 "~" H 4000 1650 50  0001 C CNN
 	1    3800 1650
@@
 AR Path="/624BFCA3/624C86EF" Ref="J9"  Part="1"
 F 0 "J9" V 2400 1200 50  0000 R CNN
-F 1 "CNX ON_OFF" V 2300 1250 50  0000 R CNN
+F 1 "ON_OFF" V 2300 1250 50  0000 R CNN
 F 2 "Connector_JST:JST_XH_B2B-XH-A_1x02_P2.50mm_Vertical" H 2200 1150 50  0001 C CNN
 F 3 "~" H 2200 1150 50  0001 C CNN
@@
 AR Path="/624BFCA3/624D4FED" Ref="TP3"  Part="1"
 F 0 "TP3" H 4150 5000 50  0000 L CNN
-F 1 "TestPoint 6V" H 4000 5100 50  0000 L CNN
-F 2 "TestPoint:TestPoint_Loop_D2.54mm_Drill1.5mm_Beaded" H 4100 4950 50  0001 C CNN
+F 1 "6V" H 4000 5100 50  0000 L CNN
+F 2 "TestPoint:TestPoint_Loop_D2.60mm_Drill1.4mm_Beaded" H 4100 4950 50  0001 C CNN
 F 3 "~" H 4100 4950 50  0001 C CNN
 	1    3900 4950
@@
 AR Path="/624BFCA3/624D5005" Ref="J13"  Part="1"
 F 0 "J13" H 4550 5700 50  0000 R CNN
-F 1 "CNX_6V" H 4600 5400 50  0000 R CNN
+F 1 "CNX 6V" H 4600 5400 50  0000 R CNN
 F 2 "TerminalBlock_Phoenix:TerminalBlock_Phoenix_MKDS-1,5-2-5.08_1x02_P5.08mm_Horizontal" H 4500 5600 50  0001 C CNN
 F 3 "~" H 4500 5600 50  0001 C CNN
@@
 AR Path="/624BFCA3/624D500B" Ref="J14"  Part="1"
 F 0 "J14" H 8850 5550 50  0000 L CNN
-F 1 "CNX_12V" H 8750 5250 50  0000 L CNN
+F 1 "CNX 12V" H 8750 5250 50  0000 L CNN
 F 2 "TerminalBlock_MetzConnect:TerminalBlock_MetzConnect_Type011_RT05502HBWC_1x02_P5.00mm_Horizontal" H 8900 5450 50  0001 C CNN
 F 3 "~" H 8900 5450 50  0001 C CNN
@@
 AR Path="/624BFCA3/624D5050" Ref="TP4"  Part="1"
 F 0 "TP4" H 8550 4900 50  0000 L CNN
-F 1 "TestPoint 12V" H 8400 5000 50  0000 L CNN
-F 2 "TestPoint:TestPoint_Loop_D2.54mm_Drill1.5mm_Beaded" H 8500 4850 50  0001 C CNN
+F 1 "12V" H 8400 5000 50  0000 L CNN
+F 2 "TestPoint:TestPoint_Loop_D2.60mm_Drill1.4mm_Beaded" H 8500 4850 50  0001 C CNN
 F 3 "~" H 8500 4850 50  0001 C CNN
 	1    8300 4850

Commit message: PCB routing completed
Connections:
- net VSS: now reaches J6.2 (Pin_2), J9.1 (Pin_1)
Changed lines of the file:
@@
 	1950 2500 2200 2500
 Wire Wire Line
-	2200 2500 2200 1350
+	2200 2500 2200 1550
 Wire Wire Line
 	2650 2750 2650 2700
@@
 	1    0    0    -1
 $EndComp
+$Comp
+L power:PWR_FLAG #FLG?
+U 1 1 62575958
+P 2150 1550
+AR Path="/62575958" Ref="#FLG?"  Part="1"
+AR Path="/624BFCA3/62575958" Ref="#FLG?"  Part="1"
+F 0 "#FLG?" H 2150 1625 50  0001 C CNN
+F 1 "PWR_FLAG" V 2150 1850 50  0000 C CNN
+F 2 "" H 2150 1550 50  0001 C CNN
+F 3 "~" H 2150 1550 50  0001 C CNN
+	1    2150 1550
+	0    -1   -1   0
+$EndComp
+Wire Wire Line
+	2150 1550 2200 1550
+Connection ~ 2200 1550
+Wire Wire Line
+	2200 1550 2200 1350
+Text Label 2000 2500 0    50   ~ 0
+VSS
 $EndSCHEMATC

Commit message: update
Parts:
- J6: value CNX POWER -> POWER IN
Changed lines of the file:
@@
 AR Path="/624BFCA3/624C86E9" Ref="J6"  Part="1"
 F 0 "J6" H 1668 2275 50  0000 C CNN
-F 1 "CNX POWER" H 1668 2366 50  0000 C CNN
+F 1 "POWER IN" H 1668 2366 50  0000 C CNN
 F 2 "TerminalBlock_Phoenix:TerminalBlock_Phoenix_MKDS-1,5-2-5.08_1x02_P5.08mm_Horizontal" H 1750 2600 50  0001 C CNN
 F 3 "~" H 1750 2600 50  0001 C CNN
